Commit message: clean

File: urdf/robot6.urdf (robot description, URDF)
Before this commit: robot m2wr, 12 links, 11 joints
Joints:
- joint camera_joint: origin xyz=0.28 0 2 rpy=0 0 0 -> xyz=0 0 0 rpy=0 0 1.57 ; parent base_link -> cluedo_link
- joint joint_laser: origin xyz=0.3 0 1 rpy=0 0 0 -> xyz=0.3 0 0.05 rpy=0 0 0

Commit message: manca poco

File: urdf/robot6.urdf (robot description, URDF)
Before this commit: robot m2wr, 12 links, 11 joints
Links:
- link left_grip_link: geometry collision box size=0.06 0.02 0.08; visual box size=0.006 0.002 0.008
- link right_grip_link: geometry collision box size=0.06 0.02 0.08; visual box size=0.006 0.002 0.008
